Commit message: created a new body for the robot

File: body.urdf (robot description, URDF)
Before this commit: robot robot, 9 links, 8 joints
Links:
- removed link BackLeg
- removed link BackLowerLeg
- removed link FrontLeg
- removed link FrontLowerLeg
- removed link LeftLeg
- removed link LeftLowerLeg
- removed link RightLeg
- removed link RightLowerLeg
- added link BackLeftLeg, mass 1; collision box size=1 0.2 0.2; visual box size=1 0.2 0.2
- added link BackLeftLowerLeg, mass 1; collision box size=0.2 0.2 1; visual box size=0.2 0.2 1
- added link BackRightLeg, mass 1; collision box size=1 0.2 0.2; visual box size=1 0.2 0.2
- added link BackRightLowerLeg, mass 1; collision box size=0.2 0.2 1; visual box size=0.2 0.2 1
- added link FrontLeftLeg, mass 1; collision box size=1 0.2 0.2; visual box size=1 0.2 0.2
- added link FrontLeftLowerLeg, mass 1; collision box size=0.2 0.2 1; visual box size=0.2 0.2 1
- added link FrontRightLeg, mass 1; collision box size=1 0.2 0.2; visual box size=1 0.2 0.2
- added link FrontRightLowerLeg, mass 1; collision box size=0.2 0.2 1; visual box size=0.2 0.2 1
- link Torso: geometry collision box size=2.5 1 1; visual box size=2.5 1 1
Joints:
- removed joint BackLeg_BackLowerLeg
- removed joint FrontLeg_FrontLowerLeg
- removed joint LeftLeg_LeftLowerLeg
- removed joint RightLeg_RightLowerLeg
- removed joint Torso_BackLeg
- removed joint Torso_FrontLeg
- removed joint Torso_LeftLeg
- removed joint Torso_RightLeg
- added joint BackLeftLeg_BackLeftLowerLeg: type revolute, parent BackLeftLeg, child BackLeftLowerLeg, origin xyz=0.9 -0.1 0 rpy=0 0 0, axis 0 1 0, limit lower=-3.14159 upper=3.14159 effort=0.0 velocity=0.0
- added joint BackRightLeg_BackRightLowerLeg: type revolute, parent BackRightLeg, child BackRightLowerLeg, origin xyz=0.9 0.1 0 rpy=0 0 0, axis 0 1 0, limit lower=-3.14159 upper=3.14159 effort=0.0 velocity=0.0
- added joint FrontLeftLeg_FrontLeftLowerLeg: type revolute, parent FrontLeftLeg, child FrontLeftLowerLeg, origin xyz=-0.9 -0.1 0 rpy=0 0 0, axis 0 1 0, limit lower=-3.14159 upper=3.14159 effort=0.0 velocity=0.0
- added joint FrontRightLeg_FrontRightLowerLeg: type revolute, parent FrontRightLeg, child FrontRightLowerLeg, origin xyz=-0.9 0.1 0 rpy=0 0 0, axis 0 1 0, limit lower=-3.14159 upper=3.14159 effort=0.0 velocity=0.0
- added joint Torso_BackLeftLeg: type revolute, parent Torso, child BackLeftLeg, origin xyz=0.75 -0.5 1 rpy=0 0 0, axis 0 1 0, limit lower=-3.14159 upper=3.14159 effort=0.0 velocity=0.0
- added joint Torso_BackRightLeg: type revolute, parent Torso, child BackRightLeg, origin xyz=0.75 0.5 1 rpy=0 0 0, axis 0 1 0, limit lower=-3.14159 upper=3.14159 effort=0.0 velocity=0.0
- added joint Torso_FrontLeftLeg: type revolute, parent Torso, child FrontLeftLeg, origin xyz=-0.75 -0.5 1 rpy=0 0 0, axis 0 1 0, limit lower=-3.14159 upper=3.14159 effort=0.0 velocity=0.0
- added joint Torso_FrontRightLeg: type revolute, parent Torso, child FrontRightLeg, origin xyz=-0.75 0.5 1 rpy=0 0 0, axis 0 1 0, limit lower=-3.14159 upper=3.14159 effort=0.0 velocity=0.0

Commit message: linked front legs and back legs together (revert to commented out lines in solution.py to undo)

File: body.urdf (robot description, URDF)
Before this commit: robot robot, 9 links, 8 joints
Links:
- link Torso: geometry collision box size=2 1 0.75; visual box size=2 1 0.75
Joints:
- joint Torso_BackLeftLeg: origin xyz=0.75 -0.5 1 rpy=0 0 0 -> xyz=0.5 -0.5 1 rpy=0 0 0
- joint Torso_BackRightLeg: origin xyz=0.75 0.5 1 rpy=0 0 0 -> xyz=0.5 0.5 1 rpy=0 0 0
- joint Torso_FrontLeftLeg: origin xyz=-0.75 -0.5 1 rpy=0 0 0 -> xyz=-0.5 -0.5 1 rpy=0 0 0
- joint Torso_FrontRightLeg: origin xyz=-0.75 0.5 1 rpy=0 0 0 -> xyz=-0.5 0.5 1 rpy=0 0 0

Commit message: added legs and head

File: body.urdf (robot description, URDF)
Before this commit: robot robot, 9 links, 8 joints
Links:
- added link Head, mass 1; collision box size=0.8 0.8 0.6; visual box size=0.8 0.8 0.6
- added link HeadLeftLeg, mass 1; collision box size=1 0.2 0.2; visual box size=1 0.2 0.2
- added link HeadLeftLowerLeg, mass 1; collision box size=0.2 0.2 1; visual box size=0.2 0.2 1
- added link HeadRightLeg, mass 1; collision box size=1 0.2 0.2; visual box size=1 0.2 0.2
- added link HeadRightLowerLeg, mass 1; collision box size=0.2 0.2 1; visual box size=0.2 0.2 1
- link Torso: geometry collision box size=1 1.5 0.75; visual box size=1 1.5 0.75
Joints:
- added joint HeadLeftLeg_HeadLeftLowerLeg: type revolute, parent HeadLeftLeg, child HeadLeftLowerLeg, origin xyz=-0.9 -0.1 0 rpy=0 0 0, axis 0 1 0, limit lower=-3.14159 upper=3.14159 effort=0.0 velocity=0.0
- added joint HeadRightLeg_HeadRightLowerLeg: type revolute, parent HeadRightLeg, child HeadRightLowerLeg, origin xyz=-0.9 0.1 0 rpy=0 0 0, axis 0 1 0, limit lower=-3.14159 upper=3.14159 effort=0.0 velocity=0.0
- added joint Head_HeadLeftLeg: type revolute, parent Head, child HeadLeftLeg, origin xyz=-0.4 -0.4 0 rpy=0 0 0, axis 0 1 0, limit lower=-3.14159 upper=3.14159 effort=0.0 velocity=0.0
- added joint Head_HeadRightLeg: type revolute, parent Head, child HeadRightLeg, origin xyz=-0.4 0.4 0 rpy=0 0 0, axis 0 1 0, limit lower=-3.14159 upper=3.14159 effort=0.0 velocity=0.0
- added joint Torso_Head: type revolute, parent Torso, child Head, origin xyz=-0.5 0 1 rpy=0 0 0, axis 0 1 0, limit lower=-3.14159 upper=3.14159 effort=0.0 velocity=0.0
- joint Torso_BackLeftLeg: origin xyz=0.5 -0.5 1 rpy=0 0 0 -> xyz=0.25 -0.75 1 rpy=0 0 0
- joint Torso_BackRightLeg: origin xyz=0.5 0.5 1 rpy=0 0 0 -> xyz=0.25 0.75 1 rpy=0 0 0
- joint Torso_FrontLeftLeg: origin xyz=-0.5 -0.5 1 rpy=0 0 0 -> xyz=-0.25 -0.75 1 rpy=0 0 0
- joint Torso_FrontRightLeg: origin xyz=-0.5 0.5 1 rpy=0 0 0 -> xyz=-0.25 0.75 1 rpy=0 0 0

Commit message: creates a snake with a random number of uniform links

File: body.urdf (robot description, URDF)
Before this commit: robot robot, 14 links, 13 joints
Links:
- removed link BackLeftLeg
- removed link BackLeftLowerLeg
- removed link BackRightLeg
- removed link BackRightLowerLeg
- removed link FrontLeftLeg
- removed link FrontLeftLowerLeg
- removed link FrontRightLeg
- removed link FrontRightLowerLeg
- removed link Head
- removed link HeadLeftLeg
- removed link HeadLeftLowerLeg
- removed link HeadRightLeg
- removed link HeadRightLowerLeg
- removed link Torso
- added link Base, mass 1; collision box size=1 1 1; visual box size=1 1 1
- added link Link0, mass 1; collision box size=1 1 1; visual box size=1 1 1
- added link Link1, mass 1; collision box size=1 1 1; visual box size=1 1 1
- added link Link2, mass 1; collision box size=1 1 1; visual box size=1 1 1
- added link Link3, mass 1; collision box size=1 1 1; visual box size=1 1 1
- added link Link4, mass 1; collision box size=1 1 1; visual box size=1 1 1
- added link Link5, mass 1; collision box size=1 1 1; visual box size=1 1 1
- added link Link6, mass 1; collision box size=1 1 1; visual box size=1 1 1
- added link Link7, mass 1; collision box size=1 1 1; visual box size=1 1 1
- added link Link8, mass 1; collision box size=1 1 1; visual box size=1 1 1
Joints:
- removed joint BackLeftLeg_BackLeftLowerLeg
- removed joint BackRightLeg_BackRightLowerLeg
- removed joint FrontLeftLeg_FrontLeftLowerLeg
- removed joint FrontRightLeg_FrontRightLowerLeg
- removed joint HeadLeftLeg_HeadLeftLowerLeg
- removed joint HeadRightLeg_HeadRightLowerLeg
- removed joint Head_HeadLeftLeg
- removed joint Head_HeadRightLeg
- removed joint Torso_BackLeftLeg
- removed joint Torso_BackRightLeg
- removed joint Torso_FrontLeftLeg
- removed joint Torso_FrontRightLeg
- removed joint Torso_Head
- added joint Base_Link0: type revolute, parent Base, child Link0, origin xyz=-0.5 0 0.5 rpy=0 0 0, axis 0 1 0, limit lower=-3.14159 upper=3.14159 effort=0.0 velocity=0.0
- added joint Link0_Link1: type revolute, parent Link0, child Link1, origin xyz=-1 0 0 rpy=0 0 0, axis 0 1 0, limit lower=-3.14159 upper=3.14159 effort=0.0 velocity=0.0
- added joint Link1_Link2: type revolute, parent Link1, child Link2, origin xyz=-1 0 0 rpy=0 0 0, axis 0 1 0, limit lower=-3.14159 upper=3.14159 effort=0.0 velocity=0.0
- added joint Link2_Link3: type revolute, parent Link2, child Link3, origin xyz=-1 0 0 rpy=0 0 0, axis 0 1 0, limit lower=-3.14159 upper=3.14159 effort=0.0 velocity=0.0
- added joint Link3_Link4: type revolute, parent Link3, child Link4, origin xyz=-1 0 0 rpy=0 0 0, axis 0 1 0, limit lower=-3.14159 upper=3.14159 effort=0.0 velocity=0.0
- added joint Link4_Link5: type revolute, parent Link4, child Link5, origin xyz=-1 0 0 rpy=0 0 0, axis 0 1 0, limit lower=-3.14159 upper=3.14159 effort=0.0 velocity=0.0
- added joint Link5_Link6: type revolute, parent Link5, child Link6, origin xyz=-1 0 0 rpy=0 0 0, axis 0 1 0, limit lower=-3.14159 upper=3.14159 effort=0.0 velocity=0.0
- added joint Link6_Link7: type revolute, parent Link6, child Link7, origin xyz=-1 0 0 rpy=0 0 0, axis 0 1 0, limit lower=-3.14159 upper=3.14159 effort=0.0 velocity=0.0
- added joint Link7_Link8: type revolute, parent Link7, child Link8, origin xyz=-1 0 0 rpy=0 0 0, axis 0 1 0, limit lower=-3.14159 upper=3.14159 effort=0.0 velocity=0.0

Commit message: randomized the size of the links

File: body.urdf (robot description, URDF)
Before this commit: robot robot, 10 links, 9 joints
Links:
- removed link Link6
- removed link Link7
- removed link Link8
- link Base: geometry collision box size=1.8807760002491114 1.907833076598838 0.8837780355914607; visual box size=1.8807760002491114 1.907833076598838 0.8837780355914607
- link Link0: geometry collision box size=0.9889110661935434 1.8513416639517342 1.8000245618403239; visual box size=0.9889110661935434 1.8513416639517342 1.8000245618403239
- link Link1: geometry collision box size=1.0250360583183091 1.3856540532007984 1.7434686551382585; visual box size=1.0250360583183091 1.3856540532007984 1.7434686551382585
- link Link2: geometry collision box size=0.9486690202408452 0.7288106127883692 1.6794775820989603; visual box size=0.9486690202408452 0.7288106127883692 1.6794775820989603
- link Link3: geometry collision box size=0.5649129495031058 1.182867098811626 1.270027359567101; visual box size=0.5649129495031058 1.182867098811626 1.270027359567101
- link Link4: geometry collision box size=1.7921471521791532 1.0121931105968074 1.2836718090985455; visual box size=1.7921471521791532 1.0121931105968074 1.2836718090985455
- link Link5: geometry collision box size=0.7407340044765955 0.5114226373731924 1.7716744370115147; visual box size=0.7407340044765955 0.5114226373731924 1.7716744370115147
Joints:
- removed joint Link5_Link6
- removed joint Link6_Link7
- removed joint Link7_Link8
- joint Base_Link0: origin xyz=-0.5 0 0.5 rpy=0 0 0 -> xyz=-0.9403880001245557 0 1 rpy=0 0 0
- joint Link0_Link1: origin xyz=-1 0 0 rpy=0 0 0 -> xyz=-0.9889110661935434 0 0 rpy=0 0 0
- joint Link1_Link2: origin xyz=-1 0 0 rpy=0 0 0 -> xyz=-1.0250360583183091 0 0 rpy=0 0 0
- joint Link2_Link3: origin xyz=-1 0 0 rpy=0 0 0 -> xyz=-0.9486690202408452 0 0 rpy=0 0 0
- joint Link3_Link4: origin xyz=-1 0 0 rpy=0 0 0 -> xyz=-0.5649129495031058 0 0 rpy=0 0 0
- joint Link4_Link5: origin xyz=-1 0 0 rpy=0 0 0 -> xyz=-1.7921471521791532 0 0 rpy=0 0 0

Commit message: finished my snake with random sensor placement

File: body.urdf (robot description, URDF)
Before this commit: robot robot, 7 links, 6 joints
Links:
- removed link Link4
- removed link Link5
- link Base: geometry collision box size=1.6391386810639297 0.7733815596414777 0.9641006047475003; visual box size=1.6391386810639297 0.7733815596414777 0.9641006047475003
- link Link0: geometry collision box size=1.7228743994019609 1.6001582664392646 1.4191349736437167; visual box size=1.7228743994019609 1.6001582664392646 1.4191349736437167
- link Link1: geometry collision box size=1.1636805441089324 0.9931075077408154 1.966871036513703; visual box size=1.1636805441089324 0.9931075077408154 1.966871036513703
- link Link2: geometry collision box size=1.7064993244535038 1.368593247869251 1.8853233962107545; visual box size=1.7064993244535038 1.368593247869251 1.8853233962107545
- link Link3: geometry collision box size=1.0567428701392694 1.5733040927860185 1.2635370427219552; visual box size=1.0567428701392694 1.5733040927860185 1.2635370427219552
Joints:
- removed joint Link3_Link4
- removed joint Link4_Link5
- joint Base_Link0: origin xyz=-0.9403880001245557 0 1 rpy=0 0 0 -> xyz=-0.8195693405319648 0 1 rpy=0 0 0
- joint Link0_Link1: origin xyz=-0.9889110661935434 0 0 rpy=0 0 0 -> xyz=-1.7228743994019609 0 0 rpy=0 0 0
- joint Link1_Link2: origin xyz=-1.0250360583183091 0 0 rpy=0 0 0 -> xyz=-1.1636805441089324 0 0 rpy=0 0 0
- joint Link2_Link3: origin xyz=-0.9486690202408452 0 0 rpy=0 0 0 -> xyz=-1.7064993244535038 0 0 rpy=0 0 0
